Commit message: fixed urdf formatting

File: src/gazebo/ros_gz_description/models/master_ASM/urdf/master_ASM.urdf (robot description, URDF)
Before this commit: robot Master_ASM, 10 links, 9 joints
Links:
- link camera_link: geometry collision mesh filename=../meshes/zed2i.stl; visual mesh filename=../meshes/zed2i.stl
